File: Senior Design/Octal_Reactor_Core/Octal_Reactor_Core_v0.sch (EAGLE design)
At the start: 61 parts, among them J1 1981584-1, SW1 EG1319, U2 MK20DX256VLH7, U3 MINI54TAN, U5 MCP73831T-2ACI/OT, Y1 32.768kHz (535-9166-2-ND), Y2 16Mhz/8pF, Y3 32.768KHz, Y4 32.768kHz

Commit message: Added Experimental Boards/ Gravity Board/ Home Automation Boards
Other:
- note added: "INERTIAL MEASUREMENT UNIT"
Changed lines of the file:
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@@
 <?xml version="1.0" encoding="utf-8"?>
 <!DOCTYPE eagle SYSTEM "eagle.dtd">
-<eagle version="9.0.1">
+<eagle version="8.7.1">
 <drawing>
 <settings>
@@
 1200mAh
 503365 Li-ion</text>
+<text x="254" y="180.34" size="2.54" layer="94">INERTIAL MEASUREMENT UNIT</text>
 </plain>
 <instances>
